Commit message: feat: add robot description

File: alpha_description/urdf/base.urdf.xacro (robot description, xacro)
@@ -3,15 +3,63 @@
     <link name="base_link">
         <visual>
-            <origin rpy="0.0 0.0 1.5707963267948966"/>
+            <origin xyz="-0.045 0.0 -0.13" rpy="0.0 1.57079632679 1.57079632679"/>
             <geometry>
-                <mesh filename="package://alpha_description/mesh/alpha.dae" scale="0.001 0.001 0.001"/>
+                <mesh filename="package://alpha_description/mesh/alpha.stl" scale="0.001 0.001 0.001"/>
             </geometry>
         </visual>
     </link>
-    <link name="imu_link"></link>
+    <link name="imu"></link>
+    <link name="imu_filter"></link>
     <joint name="imu_joint" type="fixed">
-        <origin xyz="0 0 0" rpy="0 0 0"/>
+        <origin xyz="0.0465 0.060 -0.14648" rpy="0 0 0"/>
         <parent link="base_link"/>
-        <child link="imu_link"/>
+        <child link="imu"/>
+    </joint>
+    <joint name="imu_filter_joint" type="fixed">
+        <origin xyz="0.0 0.0 0.0" rpy="0 0 0"/>
+        <parent link="imu"/>
+        <child link="imu_filter"/>
+    </joint>
+    <link name="gps"></link>
+    <joint name="gps_joint" type="fixed">
+        <origin xyz="-0.110 0.0 -0.337241" rpy="0 0 0"/>
+        <parent link="base_link"/>
+        <child link="gps"/>
+    </joint>
+    <link name="pressure"></link>
+    <joint name="pressure_joint" type="fixed">
+        <origin xyz="-0.087845 0.060 -0.124465" rpy="0 0 0"/>
+        <parent link="base_link"/>
+        <child link="pressure"/>
+    </joint>
+    <link name="dvl"></link>
+    <link name="dvl_altitude"></link>
+    <joint name="dvl_joint" type="fixed">
+        <origin xyz="0.0 0.0 0.0" rpy="0 0 0"/>
+        <parent link="base_link"/>
+        <child link="dvl"/>
+    </joint>
+    <joint name="dvl_altitude_joint" type="fixed">
+        <origin xyz="0.0 0.0 0.0" rpy="0 0 0"/>
+        <parent link="dvl"/>
+        <child link="dvl_altitude"/>
+    </joint>
+    <link name="stern_thruster_link"></link>
+    <joint name="stern_thruster_joint" type="fixed">
+        <origin xyz="-0.297 0.0 -0.130" rpy="0 0 0"/>
+        <parent link="base_link"/>
+        <child link="stern_thruster_link"/>
+    </joint>
+    <link name="vertical_thruster_link"></link>
+    <joint name="vertical_thruster_joint" type="fixed">
+        <origin xyz="0.612 0.0 -0.029" rpy="0 0 0"/>
+        <parent link="base_link"/>
+        <child link="vertical_thruster_link"/>
+    </joint>
+    <link name="horizontal_thruster_link"></link>
+    <joint name="horizontal_thruster_joint" type="fixed">
+        <origin xyz="0.691 -0.118 -0.125" rpy="0 0 0"/>
+        <parent link="base_link"/>
+        <child link="horizontal_thruster_link"/>
     </joint>
 </robot>

Commit message: fix: altitude message

File: alpha_description/urdf/base.urdf.xacro (robot description, xacro)
@@ -41,5 +41,5 @@
     </joint>
     <joint name="dvl_altitude_joint" type="fixed">
-        <origin xyz="0.0 0.0 0.0" rpy="0 0 0"/>
+        <origin xyz="0.0 0.0 0.0" rpy="0 -1.57079632679 0"/>
         <parent link="dvl"/>
         <child link="dvl_altitude"/>

Commit message: feat: add center of gravity link

File: alpha_description/urdf/base.urdf.xacro (robot description, xacro)
@@ -9,6 +9,11 @@
         </visual>
     </link>
-    <link name="imu"></link>
-    <link name="imu_filter"></link>
+    <link name="cg_link"/>
+    <joint name="cg_joint" type="fixed">
+        <origin xyz="0.223 0.000 -0.11" rpy="0 0 0"/>
+        <parent link="base_link"/>
+        <child link="cg_link"/>
+    </joint>
+    <link name="imu"/>
     <joint name="imu_joint" type="fixed">
         <origin xyz="0.0465 0.060 -0.14648" rpy="0 0 0"/>
@@ -16,4 +21,5 @@
         <child link="imu"/>
     </joint>
+    <link name="imu_filter"/>
     <joint name="imu_filter_joint" type="fixed">
         <origin xyz="0.0 0.0 0.0" rpy="0 0 0"/>
@@ -21,5 +27,5 @@
         <child link="imu_filter"/>
     </joint>
-    <link name="gps"></link>
+    <link name="gps"/>
     <joint name="gps_joint" type="fixed">
         <origin xyz="-0.110 0.0 -0.337241" rpy="0 0 0"/>
@@ -27,5 +33,5 @@
         <child link="gps"/>
     </joint>
-    <link name="pressure"></link>
+    <link name="pressure"/>
     <joint name="pressure_joint" type="fixed">
         <origin xyz="-0.087845 0.060 -0.124465" rpy="0 0 0"/>
@@ -33,6 +39,5 @@
         <child link="pressure"/>
     </joint>
-    <link name="dvl"></link>
-    <link name="dvl_altitude"></link>
+    <link name="dvl"/>
     <joint name="dvl_joint" type="fixed">
         <origin xyz="0.0 0.0 0.0" rpy="0 0 0"/>
@@ -40,4 +45,5 @@
         <child link="dvl"/>
     </joint>
+    <link name="dvl_altitude"/>
     <joint name="dvl_altitude_joint" type="fixed">
         <origin xyz="0.0 0.0 0.0" rpy="0 -1.57079632679 0"/>
@@ -45,19 +51,19 @@
         <child link="dvl_altitude"/>
     </joint>
-    <link name="stern_thruster_link"></link>
-    <joint name="stern_thruster_joint" type="fixed">
-        <origin xyz="-0.297 0.0 -0.130" rpy="0 0 0"/>
+    <link name="main_thruster_link"/>
+    <joint name="main_thruster_joint" type="fixed">
+        <origin xyz="-0.297 0.0 -0.130" rpy="0.0 0.0 0.0"/>
         <parent link="base_link"/>
-        <child link="stern_thruster_link"/>
+        <child link="main_thruster_link"/>
     </joint>
-    <link name="vertical_thruster_link"></link>
+    <link name="vertical_thruster_link"/>
     <joint name="vertical_thruster_joint" type="fixed">
-        <origin xyz="0.612 0.0 -0.029" rpy="0 0 0"/>
+        <origin xyz="0.612 0.0 -0.029" rpy="0.0 1.57079632679 0.0"/>
         <parent link="base_link"/>
         <child link="vertical_thruster_link"/>
     </joint>
-    <link name="horizontal_thruster_link"></link>
+    <link name="horizontal_thruster_link"/>
     <joint name="horizontal_thruster_joint" type="fixed">
-        <origin xyz="0.691 -0.118 -0.125" rpy="0 0 0"/>
+        <origin xyz="0.691 -0.118 -0.125" rpy="0.0 0.0 1.57079632679"/>
         <parent link="base_link"/>
         <child link="horizontal_thruster_link"/>

Commit message: feat: first working localization stack

File: alpha_description/urdf/base.urdf.xacro (robot description, xacro)
@@ -21,10 +21,4 @@
         <child link="imu"/>
     </joint>
-    <link name="imu_filter"/>
-    <joint name="imu_filter_joint" type="fixed">
-        <origin xyz="0.0 0.0 0.0" rpy="0 0 0"/>
-        <parent link="imu"/>
-        <child link="imu_filter"/>
-    </joint>
     <link name="gps"/>
     <joint name="gps_joint" type="fixed">
@@ -41,5 +35,5 @@
     <link name="dvl"/>
     <joint name="dvl_joint" type="fixed">
-        <origin xyz="0.0 0.0 0.0" rpy="0 0 0"/>
+        <origin xyz="0.0 0.0 0.0" rpy="0 0 3.14159265359"/>
         <parent link="base_link"/>
         <child link="dvl"/>

Commit message: feat: add usb cam

File: alpha_description/urdf/base.urdf.xacro (robot description, xacro)
@@ -33,4 +33,10 @@
         <child link="pressure"/>
     </joint>
+    <link name="usb_cam"/>
+    <joint name="usb_cam_joint" type="fixed">
+        <origin xyz="0.0 0.0 0.0" rpy="0 0 3.14159265359"/>
+        <parent link="base_link"/>
+        <child link="usb_cam"/>
+    </joint>
     <link name="dvl"/>
     <joint name="dvl_joint" type="fixed">

Commit message: fix: depth sensor localization fuse

File: alpha_description/urdf/base.urdf.xacro (robot description, xacro)
@@ -29,5 +29,6 @@
     <link name="pressure"/>
     <joint name="pressure_joint" type="fixed">
-        <origin xyz="-0.087845 0.060 -0.124465" rpy="0 0 0"/>
+        <origin xyz="-0.087845 0.060 -0.124465" rpy="0 3.14159265359 0"/>
+        <!--origin xyz="-0.087845 0.060 -0.124465" rpy="0.0 0.0 0.0"/-->
         <parent link="base_link"/>
         <child link="pressure"/>

Commit message: fix: thruster configuration

File: alpha_description/urdf/base.urdf.xacro (robot description, xacro)
@@ -42,5 +42,5 @@
     <link name="dvl"/>
     <joint name="dvl_joint" type="fixed">
-        <origin xyz="0.0 0.0 0.0" rpy="0 0 3.14159265359"/>
+        <origin xyz="0.0 0.0 0.0" rpy="0 0 0"/>
         <parent link="base_link"/>
         <child link="dvl"/>
@@ -60,5 +60,5 @@
     <link name="vertical_thruster_link"/>
     <joint name="vertical_thruster_joint" type="fixed">
-        <origin xyz="0.612 0.0 -0.029" rpy="0.0 1.57079632679 0.0"/>
+        <origin xyz="0.612 0.0 -0.029" rpy="0.0 -1.57079632679 0.0"/>
         <parent link="base_link"/>
         <child link="vertical_thruster_link"/>

Commit message: perf: configuration

File: alpha_description/urdf/base.urdf.xacro (robot description, xacro)
@@ -3,5 +3,5 @@
     <link name="base_link">
         <visual>
-            <origin xyz="-0.045 0.0 -0.13" rpy="0.0 1.57079632679 1.57079632679"/>
+            <origin xyz="0.0 0.0 0.0" rpy="0.0 0.0 0.0"/>
             <geometry>
                 <mesh filename="package://alpha_description/mesh/alpha.stl" scale="0.001 0.001 0.001"/>
@@ -11,5 +11,5 @@
     <link name="cg_link"/>
     <joint name="cg_joint" type="fixed">
-        <origin xyz="0.223 0.000 -0.11" rpy="0 0 0"/>
+        <origin xyz="0.100 0.000 -0.08" rpy="0 0 0"/>
         <parent link="base_link"/>
         <child link="cg_link"/>
@@ -17,5 +17,5 @@
     <link name="imu"/>
     <joint name="imu_joint" type="fixed">
-        <origin xyz="0.0465 0.060 -0.14648" rpy="0 0 0"/>
+        <origin xyz="-0.0465 -0.060 -0.14648" rpy="0 0 0"/>
         <parent link="base_link"/>
         <child link="imu"/>
@@ -23,5 +23,5 @@
     <link name="gps"/>
     <joint name="gps_joint" type="fixed">
-        <origin xyz="-0.110 0.0 -0.337241" rpy="0 0 0"/>
+        <origin xyz="-0.320 0.0 -0.437241" rpy="0 0 0"/>
         <parent link="base_link"/>
         <child link="gps"/>
@@ -29,5 +29,5 @@
     <link name="pressure"/>
     <joint name="pressure_joint" type="fixed">
-        <origin xyz="-0.087845 0.060 -0.124465" rpy="0 3.14159265359 0"/>
+        <origin xyz="-0.187845 -0.060 -0.124465" rpy="0 3.14159265359 0"/>
         <!--origin xyz="-0.087845 0.060 -0.124465" rpy="0.0 0.0 0.0"/-->
         <parent link="base_link"/>
@@ -36,5 +36,5 @@
     <link name="usb_cam"/>
     <joint name="usb_cam_joint" type="fixed">
-        <origin xyz="0.0 0.0 0.0" rpy="0 0 3.14159265359"/>
+        <origin xyz="-0.112533 0.0 0.0" rpy="0 0 3.14159265359"/>
         <parent link="base_link"/>
         <child link="usb_cam"/>
@@ -54,5 +54,5 @@
     <link name="main_thruster_link"/>
     <joint name="main_thruster_joint" type="fixed">
-        <origin xyz="-0.297 0.0 -0.130" rpy="0.0 0.0 0.0"/>
+        <origin xyz="-0.524 0.0 -0.130" rpy="0.0 0.0 0.0"/>
         <parent link="base_link"/>
         <child link="main_thruster_link"/>
@@ -60,5 +60,5 @@
     <link name="vertical_thruster_link"/>
     <joint name="vertical_thruster_joint" type="fixed">
-        <origin xyz="0.612 0.0 -0.029" rpy="0.0 -1.57079632679 0.0"/>
+        <origin xyz="0.48735 0.0 -0.029" rpy="0.0 -1.57079632679 0.0"/>
         <parent link="base_link"/>
         <child link="vertical_thruster_link"/>
@@ -66,5 +66,5 @@
     <link name="horizontal_thruster_link"/>
     <joint name="horizontal_thruster_joint" type="fixed">
-        <origin xyz="0.691 -0.118 -0.125" rpy="0.0 0.0 1.57079632679"/>
+        <origin xyz="0.57635 -0.118 -0.125" rpy="0.0 0.0 1.57079632679"/>
         <parent link="base_link"/>
         <child link="horizontal_thruster_link"/>

Commit message: fix: center of gravity position

File: alpha_description/urdf/base.urdf.xacro (robot description, xacro)
@@ -11,5 +11,5 @@
     <link name="cg_link"/>
     <joint name="cg_joint" type="fixed">
-        <origin xyz="0.100 0.000 -0.08" rpy="0 0 0"/>
+        <origin xyz="0.100 0.000 -0.10" rpy="0 0 0"/>
         <parent link="base_link"/>
         <child link="cg_link"/>

Commit message: fix: thruster configuration after maintenance

File: alpha_description/urdf/base.urdf.xacro (robot description, xacro)
@@ -60,5 +60,5 @@
     <link name="vertical_thruster_link"/>
     <joint name="vertical_thruster_joint" type="fixed">
-        <origin xyz="0.48735 0.0 -0.029" rpy="0.0 -1.57079632679 0.0"/>
+        <origin xyz="0.48735 0.0 -0.029" rpy="0.0 1.57079632679 0.0"/>
         <parent link="base_link"/>
         <child link="vertical_thruster_link"/>

Commit message: fix: config

File: alpha_description/urdf/base.urdf.xacro (robot description, xacro)
@@ -66,5 +66,5 @@
     <link name="horizontal_thruster_link"/>
     <joint name="horizontal_thruster_joint" type="fixed">
-        <origin xyz="0.57635 -0.118 -0.125" rpy="0.0 0.0 1.57079632679"/>
+        <origin xyz="0.57635 -0.118 -0.125" rpy="0.0 0.0 -1.57079632679"/>
         <parent link="base_link"/>
         <child link="horizontal_thruster_link"/>
