Commit message: fix: localization

File: alpha_description/urdf/base_v1-1.urdf.xacro (robot description, xacro)
@@ -3,5 +3,5 @@
     <link name="base_link">
         <visual>
-            <origin xyz="0.155 0.0 -0.65" rpy="-1.571 0.0 3.1415"/>
+            <origin xyz="0.155 0.0 0.65" rpy="1.571 0.0 3.1415"/>
             <geometry>
                 <mesh filename="package://alpha_description/mesh/alpha_v1-1.stl" scale="0.001 0.001 0.001"/>
@@ -11,5 +11,5 @@
     <link name="cg_link"/>
     <joint name="cg_joint" type="fixed">
-        <origin xyz="0.100 0.000 -0.10" rpy="0 0 0"/>
+        <origin xyz="0.100 0.000 0.10" rpy="3.14159265359 0.0 0.0"/>
         <parent link="base_link"/>
         <child link="cg_link"/>
@@ -17,5 +17,5 @@
     <link name="imu"/>
     <joint name="imu_joint" type="fixed">
-        <origin xyz="-0.0465 -0.060 -0.14648" rpy="0 0 0"/>
+        <origin xyz="-0.0465 0.060 0.14648" rpy="3.14159265359 0.0 0.0"/>
         <parent link="base_link"/>
         <child link="imu"/>
@@ -23,5 +23,5 @@
     <link name="gps"/>
     <joint name="gps_joint" type="fixed">
-        <origin xyz="0.1 0.0 -0.407241" rpy="0 0 0"/>
+        <origin xyz="0.1 0.0 0.407241" rpy="0.0 0.0 0.0"/>
         <parent link="base_link"/>
         <child link="gps"/>
@@ -29,5 +29,5 @@
     <link name="pressure"/>
     <joint name="pressure_joint" type="fixed">
-        <origin xyz="-0.187845 -0.060 -0.124465" rpy="0 3.14159265359 0"/>
+        <origin xyz="-0.187845 -0.060 0.124465" rpy="0.0 3.14159265359 0.0"/>
         <!--origin xyz="-0.087845 0.060 -0.124465" rpy="0.0 0.0 0.0"/-->
         <parent link="base_link"/>
@@ -36,5 +36,5 @@
     <link name="usb_cam"/>
     <joint name="usb_cam_joint" type="fixed">
-        <origin xyz="-0.112533 0.0 0.0" rpy="0 0 3.14159265359"/>
+        <origin xyz="-0.112533 0.0 0.0" rpy="0.0 0.0 3.14159265359"/>
         <parent link="base_link"/>
         <child link="usb_cam"/>
@@ -42,5 +42,5 @@
     <link name="dvl"/>
     <joint name="dvl_joint" type="fixed">
-        <origin xyz="0.0 0.0 0.0" rpy="0 0 0"/>
+        <origin xyz="0.0 0.0 0.0" rpy="3.14159265359 0 0"/>
         <parent link="base_link"/>
         <child link="dvl"/>
@@ -48,5 +48,5 @@
     <link name="dvl_altitude"/>
     <joint name="dvl_altitude_joint" type="fixed">
-        <origin xyz="0.0 0.0 0.0" rpy="0 -1.57079632679 0"/>
+        <origin xyz="0.0 0.0 0.0" rpy="0 1.57079632679 0"/>
         <parent link="dvl"/>
         <child link="dvl_altitude"/>
@@ -54,5 +54,5 @@
     <link name="surge_thruster_link"/>
     <joint name="surge_thruster_joint" type="fixed">
-        <origin xyz="-0.554 0.0 -0.100" rpy="0.0 0.0 0.0"/>
+        <origin xyz="-0.554 0.0 0.100" rpy="0.0 0.0 0.0"/>
         <parent link="base_link"/>
         <child link="surge_thruster_link"/>
@@ -60,5 +60,5 @@
     <link name="heave_stern_thruster_link"/>
     <joint name="heave_stern_thruster_joint" type="fixed">
-        <origin xyz="0.48735 0.0 -0.089" rpy="0.0 1.57079632679 0.0"/>
+        <origin xyz="0.48735 0.0 0.089" rpy="0.0 -1.57079632679 0.0"/>
         <parent link="base_link"/>
         <child link="heave_stern_thruster_link"/>
@@ -66,5 +66,5 @@
     <link name="heave_bow_thruster_link"/>
     <joint name="heave_bow_thruster_joint" type="fixed">
-        <origin xyz="-0.28045 0.0 -0.089" rpy="0.0 1.57079632679 0.0"/>
+        <origin xyz="-0.28045 0.0 0.089" rpy="0.0 -1.57079632679 0.0"/>
         <parent link="base_link"/>
         <child link="heave_bow_thruster_link"/>
@@ -72,5 +72,5 @@
     <link name="sway_stern_thruster_link"/>
     <joint name="sway_stern_thruster_joint" type="fixed">
-        <origin xyz="0.57635 0.0 -0.105" rpy="0.0 0.0 1.57079632679"/>
+        <origin xyz="0.57635 0.0 0.105" rpy="0.0 0.0 -1.57079632679"/>
         <parent link="base_link"/>
         <child link="sway_stern_thruster_link"/>

Commit message: multibeam integrated, but minor issue with TF

File: alpha_description/urdf/base_v1-1.urdf.xacro (robot description, xacro)
@@ -76,3 +76,9 @@
         <child link="sway_stern_thruster_link"/>
     </joint>
+    <link name="multibeam"/>
+    <joint name="multibeam_joint" type="fixed">
+        <origin xyz="0.0 0.0 0.2" rpy="0.0 1.57079632679 3.1415926"/>
+        <parent link="base_link"/>
+        <child link="multibeam"/>
+    </joint>
 </robot>

Commit message: feat: separate scenario files

File: alpha_description/urdf/base_v1-1.urdf.xacro (robot description, xacro)
@@ -78,5 +78,5 @@
     <link name="multibeam"/>
     <joint name="multibeam_joint" type="fixed">
-        <origin xyz="0.0 0.0 0.2" rpy="0.0 1.57079632679 3.1415926"/>
+        <origin xyz="0.0 0.0 0.2" rpy="3.1416 1.0471975511965976 0.0"/>
         <parent link="base_link"/>
         <child link="multibeam"/>

Commit message: refactor: seal_msgs -> mvp_msgs

File: alpha_description/urdf/base_v1-1.urdf.xacro (robot description, xacro)
@@ -58,21 +58,21 @@
         <child link="surge_thruster_link"/>
     </joint>
+    <link name="heave_bow_thruster_link"/>
+    <joint name="heave_bow_thruster_joint" type="fixed">
+        <origin xyz="0.48735 0.0 0.089" rpy="0.0 -1.57079632679 0.0"/>
+        <parent link="base_link"/>
+        <child link="heave_bow_thruster_link"/>
+    </joint>
     <link name="heave_stern_thruster_link"/>
     <joint name="heave_stern_thruster_joint" type="fixed">
-        <origin xyz="0.48735 0.0 0.089" rpy="0.0 -1.57079632679 0.0"/>
+        <origin xyz="-0.28045 0.0 0.089" rpy="0.0 -1.57079632679 0.0"/>
         <parent link="base_link"/>
         <child link="heave_stern_thruster_link"/>
     </joint>
-    <link name="heave_bow_thruster_link"/>
-    <joint name="heave_bow_thruster_joint" type="fixed">
-        <origin xyz="-0.28045 0.0 0.089" rpy="0.0 -1.57079632679 0.0"/>
-        <parent link="base_link"/>
-        <child link="heave_bow_thruster_link"/>
-    </joint>
-    <link name="sway_stern_thruster_link"/>
-    <joint name="sway_stern_thruster_joint" type="fixed">
+    <link name="sway_bow_thruster_link"/>
+    <joint name="sway_bow_thruster_joint" type="fixed">
         <origin xyz="0.57635 0.0 0.105" rpy="0.0 0.0 -1.57079632679"/>
         <parent link="base_link"/>
-        <child link="sway_stern_thruster_link"/>
+        <child link="sway_bow_thruster_link"/>
     </joint>
     <link name="multibeam"/>

Commit message: config: update configuration based on the platform

File: alpha_description/urdf/base_v1-1.urdf.xacro (robot description, xacro)
@@ -60,5 +60,5 @@
     <link name="heave_bow_thruster_link"/>
     <joint name="heave_bow_thruster_joint" type="fixed">
-        <origin xyz="0.48735 0.0 0.089" rpy="0.0 -1.57079632679 0.0"/>
+        <origin xyz="0.48735 0.0 0.089" rpy="0.0 1.57079632679 0.0"/>
         <parent link="base_link"/>
         <child link="heave_bow_thruster_link"/>
@@ -66,5 +66,5 @@
     <link name="heave_stern_thruster_link"/>
     <joint name="heave_stern_thruster_joint" type="fixed">
-        <origin xyz="-0.28045 0.0 0.089" rpy="0.0 -1.57079632679 0.0"/>
+        <origin xyz="-0.28045 0.0 0.089" rpy="0.0 1.57079632679 0.0"/>
         <parent link="base_link"/>
         <child link="heave_stern_thruster_link"/>
@@ -72,5 +72,5 @@
     <link name="sway_bow_thruster_link"/>
     <joint name="sway_bow_thruster_joint" type="fixed">
-        <origin xyz="0.57635 0.0 0.105" rpy="0.0 0.0 -1.57079632679"/>
+        <origin xyz="0.57635 0.0 0.105" rpy="0.0 0.0 1.57079632679"/>
         <parent link="base_link"/>
         <child link="sway_bow_thruster_link"/>

Commit message: tf between base_link and sidescan

File: alpha_description/urdf/base_v1-1.urdf.xacro (robot description, xacro)
@@ -78,7 +78,33 @@
     <link name="multibeam"/>
     <joint name="multibeam_joint" type="fixed">
-        <origin xyz="0.0 0.0 0.2" rpy="3.1416 1.0471975511965976 0.0"/>
+        <origin xyz="0.0 0.0 -0.2" rpy="3.1416 1.0471975511965976 0.0"/>
         <parent link="base_link"/>
         <child link="multibeam"/>
     </joint>
+    <!-- TF between Base frame and Transducer frame -->
+    <link name="ifss_port"/>
+    <joint name="ifss_port_joint" type="fixed">
+        <origin xyz="0 0.0762 -0.2" rpy="-1.5708 0.523599 1.5708"/>
+        <parent link="base_link"/>
+        <child link="ifss_port"/>
+    </joint>
+    <link name="ifss_starboard"/>
+    <joint name="ifss_starboard_joint" type="fixed">
+        <origin xyz="0 -0.0762 -0.2" rpy="1.5708 0.523599 -1.5708"/>
+        <parent link="base_link"/>
+        <child link="ifss_starboard"/>
+    </joint>
+    <!-- TF between Transducer frame and Swath frame -->
+    <link name="ifss_port_swath"/>
+    <joint name="ifss_port_swath_joint" type="fixed">
+        <origin xyz="0 0 0" rpy="0 0 0.261799383"/>
+        <parent link="ifss_port"/>
+        <child link="ifss_port_swath"/>
+    </joint>
+    <link name="ifss_starboard_swath"/>
+    <joint name="ifss_starboard_swath_joint" type="fixed">
+        <origin xyz="0 0 0" rpy="0 0 -0.261799383"/>
+        <parent link="ifss_starboard"/>
+        <child link="ifss_starboard_swath"/>
+    </joint>
 </robot>

Commit message: fix: global localization

File: alpha_description/urdf/base_v1-1.urdf.xacro (robot description, xacro)
@@ -23,5 +23,5 @@
     <link name="gps"/>
     <joint name="gps_joint" type="fixed">
-        <origin xyz="0.1 0.0 0.407241" rpy="0.0 0.0 0.0"/>
+        <origin xyz="0.1 0.0 0.407241" rpy="3.1415 0.0 0.0"/>
         <parent link="base_link"/>
         <child link="gps"/>

Commit message: docs: update file descriptions and readme

File: alpha_description/urdf/base_v1-1.urdf.xacro (robot description, xacro)
@@ -42,5 +42,5 @@
     <link name="dvl"/>
     <joint name="dvl_joint" type="fixed">
-        <origin xyz="0.0 0.0 0.0" rpy="3.14159265359 0 0"/>
+        <origin xyz="0.0 0.0 0.0" rpy="0.0 0.0 0.0"/>
         <parent link="base_link"/>
         <child link="dvl"/>
