Commit message: feat: add namespaces

File: alpha_stonefish/description/alpha.scn.xacro (robot description, xacro)
@@ -7,8 +7,9 @@
     Copyright (C) 2022 Smart Ocean Systems Laboratory
 -->
-<scenario>
-    <include file="$(find alpha_stonefish)/description/looks.scn"/>
-    <include file="$(find alpha_stonefish)/description/materials.scn"/>
-    <robot name="alpha" fixed="false" self_collisions="false">
+<scenario xmlns:xacro="http://ros.org/wiki/xacro">
+    <xacro:arg name="robot_name" default="changeme"/>
+    <xacro:include filename="$(find alpha_stonefish)/description/looks.scn.xacro"/>
+    <xacro:include filename="$(find alpha_stonefish)/description/materials.scn.xacro"/>
+    <robot name="$(arg robot_name)" fixed="false" self_collisions="false">
         <base_link name="Vehicle" type="compound" physics="submerged">
             <external_part name="Hull" type="model" physics="submerged" buoyant="false">
@@ -71,5 +72,5 @@
                 <look name="white"/>
             </propeller>
-            <ros_subscriber topic="/control/thruster/heave_stern"/>
+            <ros_subscriber topic="/$(arg robot_name)/control/thruster/heave_stern"/>
         </actuator>
         <actuator name="ThrusterHeaveBow" type="thruster">
@@ -82,5 +83,5 @@
                 <look name="white"/>
             </propeller>
-            <ros_subscriber topic="/control/thruster/heave_bow"/>
+            <ros_subscriber topic="/$(arg robot_name)/control/thruster/heave_bow"/>
         </actuator>
         <actuator name="ThrusterSwayBow" type="thruster">
@@ -93,5 +94,5 @@
                 <look name="white"/>
             </propeller>
-            <ros_subscriber topic="/control/thruster/sway_bow"/>
+            <ros_subscriber topic="/$(arg robot_name)/control/thruster/sway_bow"/>
         </actuator>
         <actuator name="ThrusterSurge" type="thruster">
@@ -105,5 +106,5 @@
                 <look name="white"/>
             </propeller>
-            <ros_subscriber topic="/control/thruster/surge"/>
+            <ros_subscriber topic="/$(arg robot_name)/control/thruster/surge"/>
         </actuator>
         <sensor name="pressure" type="pressure" rate="5.0">
@@ -111,5 +112,5 @@
             <origin rpy="0.0 0.0 0.0" xyz="-1.20 0.0 0.0"/>
             <noise pressure="5.0"/>
-            <ros_publisher topic="/pressure"/>
+            <ros_publisher topic="/$(arg robot_name)/pressure"/>
         </sensor>
         <sensor name="dvl" type="dvl" rate="5.0">
@@ -119,5 +120,5 @@
             <range velocity="9.0 9.0 9.0" altitude_min="0.05" altitude_max="200.0"/>
             <noise velocity="0.0015" altitude="0.001"/>
-            <ros_publisher topic="/dvl/twist" altitude_topic="/dvl/altitude"/>
+            <ros_publisher topic="/$(arg robot_name)/dvl/twist" altitude_topic="/$(arg robot_name)/dvl/altitude"/>
         </sensor>
         <sensor name="imu" type="imu" rate="20.0">
@@ -125,5 +126,5 @@
             <origin rpy="0.0 0.0 0.0" xyz="-0.65 0.0 0.0"/>
             <noise angle="0.000001745" angular_velocity="0.00001745"/>
-            <ros_publisher topic="/imu/stonefish/data"/>
+            <ros_publisher topic="/$(arg robot_name)/imu/stonefish/data"/>
         </sensor>
         <sensor name="gps" type="gps" rate="1.0">
@@ -131,5 +132,5 @@
             <origin rpy="0.0 0.0 0.0" xyz="-0.54 0.0 -0.2"/>
             <noise ned_position="0.5"/>
-            <ros_publisher topic="/gps/fix"/>
+            <ros_publisher topic="/$(arg robot_name)/gps/fix"/>
         </sensor>
         <sensor name="multibeam" rate="50.0" type="multibeam">
@@ -140,15 +141,6 @@
             <origin xyz="0.0 0.0 0.2" rpy="0.0 -1.0471975511965976 0.0"/>
             <link name="Vehicle"/>
-            <ros_publisher topic="/mbs/data"/>
+            <ros_publisher topic="/$(arg robot_name)/mbs/data"/>
         </sensor>
-        <!-- <sensor name="MSIS" type="msis">
-            <link name="Vehicle"/>
-            <specs step="1.0" bins="500" horizontal_beam_width="2.0" vertical_beam_width="2.0"/>
-            <settings range_min="0.5" range_max="50.0" rotation_min="-180.0" rotation_max="180.0" gain="20.0"/>
-            <noise multiplicative="0.01" additive="0.01"/>
-            <display colormap="hot"/>
-            <origin xyz="0.0 0.0 0.0" rpy="1.57 0.00 1.57"/>
-            <ros_publisher topic="/msis/data"/>
-        </sensor> -->
         <sensor name="ifss_port_swath" rate="10.0" type="multibeam">
             <specs fov="53.0" steps="64"/>
@@ -158,6 +150,6 @@
             <origin xyz="-0.75 -0.0762 0.2" rpy="-1.5708 -2.35619 1.5708"/>
             <link name="Vehicle"/>
-            <pcl_topic topic="/ifss/port/pcl"/>
-            <ros_publisher topic="/ifss/port"/>
+            <pcl_topic topic="/$(arg robot_name)/ifss/port/pcl"/>
+            <ros_publisher topic="/$(arg robot_name)/ifss/port"/>
         </sensor>
         <sensor name="ifss_starboard_swath" rate="10.0" type="multibeam">
@@ -168,6 +160,6 @@
             <origin xyz="-0.75 0.0762 0.2" rpy="1.5708 -2.35619 -1.5708"/>
             <link name="Vehicle"/>
-            <pcl_topic topic="/ifss/starboard/pcl"/>
-            <ros_publisher topic="/ifss/starboard"/>
+            <pcl_topic topic="/$(arg robot_name)/ifss/starboard/pcl"/>
+            <ros_publisher topic="/$(arg robot_name)/ifss/starboard"/>
         </sensor>
         <world_transform rpy="0.0 0.0 0.0" xyz="0.0 0.0 0.0"/>

File: alpha_stonefish/scenarios/ocean.scn.xacro (robot description, xacro)
@@ -7,8 +7,9 @@
     Copyright (C) 2022 Smart Ocean Systems Laboratory
 -->
-<scenario>
-    <include file="$(find alpha_stonefish)/description/alpha.scn"/>
+<scenario xmlns:xacro="http://ros.org/wiki/xacro">
+    <xacro:arg name="robot_name" default="changeme"/>
+    <xacro:include filename="$(find alpha_stonefish)/description/alpha.scn.xacro"/>
     <environment>
-        <ned latitude="41.7777" longitude="3.0333"/>
+        <ned latitude="41" longitude="71"/>
         <ocean>
             <water density="1000.0" jerlov="0.2"/>
@@ -23,16 +24,16 @@
         </atmosphere>
     </environment>
-    <static name="tank" type="model">
+    <static name="Bottom" type="model">
         <physical>
-            <mesh filename="tank.obj" scale="1.0" convex="false"/>
+            <mesh filename="seabed.obj" scale="2.0" convex="false"/>
             <origin xyz="0.0 0.0 0.0" rpy="0.0 0.0 0.0"/>
         </physical>
         <visual>
-            <mesh filename="tank.obj" scale="1.0"/>
+            <mesh filename="seabed.obj" scale="2.0"/>
             <origin xyz="0.0 0.0 0.0" rpy="0.0 0.0 0.0"/>
         </visual>
         <material name="Rock"/>
         <look name="Gray"/>
-        <world_transform xyz="0.0 0.0 18.0" rpy="3.1415926 0.0 0.0"/>
+        <world_transform xyz="-500.0 -500.0 -130.0" rpy="0.0 0.0 0.0"/>
     </static>
 </scenario>

File: alpha_stonefish/scenarios/tank.scn.xacro (robot description, xacro)
@@ -7,8 +7,9 @@
     Copyright (C) 2022 Smart Ocean Systems Laboratory
 -->
-<scenario>
-    <include file="$(find alpha_stonefish)/description/alpha.scn"/>
+<scenario xmlns:xacro="http://ros.org/wiki/xacro">
+    <xacro:arg name="robot_name" default="changeme"/>
+    <xacro:include filename="$(find alpha_stonefish)/description/alpha.scn.xacro"/>
     <environment>
-        <ned latitude="41" longitude="71"/>
+        <ned latitude="41.7777" longitude="3.0333"/>
         <ocean>
             <water density="1000.0" jerlov="0.2"/>
@@ -23,16 +24,16 @@
         </atmosphere>
     </environment>
-    <static name="Bottom" type="model">
+    <static name="tank" type="model">
         <physical>
-            <mesh filename="seabed.obj" scale="2.0" convex="false"/>
+            <mesh filename="tank.obj" scale="1.0" convex="false"/>
             <origin xyz="0.0 0.0 0.0" rpy="0.0 0.0 0.0"/>
         </physical>
         <visual>
-            <mesh filename="seabed.obj" scale="2.0"/>
+            <mesh filename="tank.obj" scale="1.0"/>
             <origin xyz="0.0 0.0 0.0" rpy="0.0 0.0 0.0"/>
         </visual>
         <material name="Rock"/>
         <look name="Gray"/>
-        <world_transform xyz="-500.0 -500.0 -130.0" rpy="0.0 0.0 0.0"/>
+        <world_transform xyz="0.0 0.0 18.0" rpy="3.1415926 0.0 0.0"/>
     </static>
 </scenario>
