Commit message: feat: add alpha with rotating thrusters

File: alpha_stonefish/description/alpha.scn.xacro (robot description, xacro)
@@ -1,168 +1,4 @@
-<?xml version="1.0"?>
-<!--
-    This file is part of ALPHA AUV project.
-    Author: Emir Cem Gezer
-    Email: emircem@uri.edu;emircem.gezer@gmail.com
-    Year: 2022
-    Copyright (C) 2022 Smart Ocean Systems Laboratory
--->
 <scenario xmlns:xacro="http://ros.org/wiki/xacro">
-    <xacro:include filename="$(find alpha_stonefish)/description/looks.scn.xacro"/>
-    <xacro:include filename="$(find alpha_stonefish)/description/materials.scn.xacro"/>
-    <xacro:macro name="alpha" params="xyz rpy robot_name">
-        <robot name="${robot_name}" fixed="false" self_collisions="false">
-            <base_link name="Vehicle" type="compound" physics="submerged">
-                <external_part name="Hull" type="model" physics="submerged" buoyant="false">
-                    <physical>
-                        <mesh filename="hull_phy_reduced.obj" scale="1.0"/>
-                        <origin rpy="0.0 0.0 0.0" xyz="0.0 0.0 0.0"/>
-                    </physical>
-                    <visual>
-                        <mesh filename="hull.obj" scale="1.0"/>
-                        <origin rpy="0.0 0.0 0.0" xyz="0.0 0.0 0.0"/>
-                    </visual>
-                    <material name="Vehicle"/>
-                    <look name="yellow"/>
-                    <mass value="24.8"/>
-                    <compound_transform rpy="0.0 0.0 0.0" xyz="0.0 0.0 0.0"/>
-                    <cg xyz="-0.65 0.0 0.1" rpy="0.0 0.0 0.0"/>
-                </external_part>
-                <internal_part name="Foam" type="cylinder" physics="floating" buoyant="true">
-                    <dimensions radius="0.1" height="1.0"/>
-                    <origin rpy="0.0 0.0 0.0" xyz="0.0 0.0 0.0"/>
-                    <material name="Foam"/>
-                    <mass value="6.0"/>
-                    <look name="grey"/>
-                    <compound_transform rpy="0.0 1.571 0.0" xyz="-0.65 0.0 -0.05"/>
-                </internal_part>
-                <external_part name="Mast" type="model" physics="submerged">
-                    <physical>
-                        <mesh filename="mast.obj" scale="0.001"/>
-                        <origin rpy="-1.571 0.0 1.571"  xyz="-1.0 0.0 0.0"/>
-                    </physical>
-                    <visual>
-                        <mesh filename="mast.obj" scale="0.001"/>
-                        <origin rpy="-1.571 0.0 1.571" xyz="-1.0 0.0 0.0"/>
-                    </visual>
-                    <material name="Resin"/>
-                    <look name="white"/>
-                    <compound_transform rpy="0.0 0.0 0.0" xyz="0.0 0.0 0.0"/>
-                </external_part>
-                <external_part name="ThrusterDuctSurge" type="model" physics="submerged" buoyant="false">
-                    <physical>
-                        <mesh filename="duct.obj" scale="0.0015"/>
-                        <origin rpy="0.0 1.571 0.0" xyz="-1.325 0.0 0.0"/>
-                    </physical>
-                    <visual>
-                        <mesh filename="duct.obj" scale="0.0015"/>
-                        <origin rpy="0.0 1.571 0.0" xyz="-1.325 0.0 0.0"/>
-                    </visual>
-                    <material name="Neutral"/>
-                    <look name="black"/>
-                    <compound_transform rpy="0.0 0.0 0.0" xyz="0.0 0.0 0.0"/>
-                </external_part>
-            </base_link>
-            <actuator name="ThrusterHeaveStern" type="thruster">
-                <link name="Vehicle"/>
-                <origin rpy="0.0 -1.571 0.0" xyz="-1.0956 0.0 0.0"/>
-                <specs thrust_coeff="0.4315" thrust_coeff_backward="0.3404" torque_coeff="0.01" max_rpm="3000.0"/>
-                <propeller diameter="0.08" right="true">
-                    <mesh filename="prop.obj" scale="1.0"/>
-                    <material name="Neutral"/>
-                    <look name="white"/>
-                </propeller>
-                <ros_subscriber topic="/${robot_name}/control/thruster/heave_stern"/>
-            </actuator>
-            <actuator name="ThrusterHeaveBow" type="thruster">
-                <link name="Vehicle"/>
-                <origin rpy="0.0 -1.571 0.0" xyz="-0.2857 0.0 0.0"/>
-                <specs thrust_coeff="0.4315" thrust_coeff_backward="0.3404" torque_coeff="0.01" max_rpm="3000.0"/>
-                <propeller diameter="0.08" right="true">
-                    <mesh filename="prop.obj" scale="1.0"/>
-                    <material name="Neutral"/>
-                    <look name="white"/>
-                </propeller>
-                <ros_subscriber topic="/${robot_name}/control/thruster/heave_bow"/>
-            </actuator>
-            <actuator name="ThrusterSwayBow" type="thruster">
-                <link name="Vehicle"/>
-                <origin rpy="0.0 0.0 -1.571" xyz="-0.171 0.0 0.0"/>
-                <specs thrust_coeff="0.4315" thrust_coeff_backward="0.3404" torque_coeff="0.01" max_rpm="3000.0"/>
-                <propeller diameter="0.08" right="true">
-                    <mesh filename="prop.obj" scale="1.0"/>
-                    <material name="Neutral"/>
-                    <look name="white"/>
-                </propeller>
-                <ros_subscriber topic="/${robot_name}/control/thruster/sway_bow"/>
-            </actuator>
-            <actuator name="ThrusterSurge" type="thruster">
-                <link name="Vehicle"/>
-                <origin rpy="0.0 0.0 0.0" xyz="-1.325 0.0 0.0"/>
-                <specs thrust_coeff="1.7568" thrust_coeff_backward="1.0882" torque_coeff="0.01" max_rpm="3000.0"/>
-                <propeller diameter="0.08" right="true">
-                    <origin rpy="1.571 0.0 0.0" xyz="0.0 0.0 0.0"/>
-                    <mesh filename="prop.obj" scale="1.5"/>
-                    <material name="Neutral"/>
-                    <look name="white"/>
-                </propeller>
-                <ros_subscriber topic="/${robot_name}/control/thruster/surge"/>
-            </actuator>
-            <sensor name="pressure" type="pressure" rate="5.0">
-                <link name="Vehicle"/>
-                <origin rpy="0.0 0.0 0.0" xyz="-1.20 0.0 0.0"/>
-                <noise pressure="5.0"/>
-                <ros_publisher topic="/${robot_name}/pressure"/>
-            </sensor>
-            <sensor name="dvl" type="dvl" rate="5.0">
-                <link name="Vehicle"/>
-                <origin rpy="3.1416 0.0 0.0" xyz="-0.75 0.0 0.10"/>
-                <specs beam_angle="30.0"/>
-                <range velocity="9.0 9.0 9.0" altitude_min="0.05" altitude_max="200.0"/>
-                <noise velocity="0.0015" altitude="0.001"/>
-                <ros_publisher topic="/${robot_name}/dvl/twist" altitude_topic="/${robot_name}/dvl/altitude"/>
-            </sensor>
-            <sensor name="imu" type="imu" rate="20.0">
-                <link name="Vehicle"/>
-                <origin rpy="0.0 0.0 0.0" xyz="-0.65 0.0 0.0"/>
-                <noise angle="0.000001745" angular_velocity="0.00001745"/>
-                <ros_publisher topic="/${robot_name}/imu/stonefish/data"/>
-            </sensor>
-            <sensor name="gps" type="gps" rate="1.0">
-                <link name="Vehicle"/>
-                <origin rpy="0.0 0.0 0.0" xyz="-0.54 0.0 -0.2"/>
-                <noise ned_position="0.5"/>
-                <ros_publisher topic="/${robot_name}/gps/fix"/>
-            </sensor>
-            <sensor name="multibeam" rate="50.0" type="multibeam">
-                <specs fov="90.0" steps="64"/>
-                <range distance_min="0.5" distance_max="200.0"/>
-                <noise distance="0.0"/>
-                <history samples="1"/>
-                <origin xyz="0.0 0.0 0.2" rpy="0.0 -1.0471975511965976 0.0"/>
-                <link name="Vehicle"/>
-                <ros_publisher topic="/${robot_name}/mbs/data"/>
-            </sensor>
-            <sensor name="ifss_port_swath" rate="10.0" type="multibeam">
-                <specs fov="53.0" steps="64"/>
-                <range distance_min="0.1" distance_max="150.0"/>
-                <noise distance="0.0"/>
-                <history samples="1"/>
-                <origin xyz="-0.75 -0.0762 0.2" rpy="-1.5708 -2.35619 1.5708"/>
-                <link name="Vehicle"/>
-                <pcl_topic topic="/${robot_name}/ifss/port/pcl"/>
-                <ros_publisher topic="/${robot_name}/ifss/port"/>
-            </sensor>
-            <sensor name="ifss_starboard_swath" rate="10.0" type="multibeam">
-                <specs fov="53.0" steps="64"/>
-                <range distance_min="0.1" distance_max="150.0"/>
-                <noise distance="0.0"/>
-                <history samples="1"/>
-                <origin xyz="-0.75 0.0762 0.2" rpy="1.5708 -2.35619 -1.5708"/>
-                <link name="Vehicle"/>
-                <pcl_topic topic="/${robot_name}/ifss/starboard/pcl"/>
-                <ros_publisher topic="/${robot_name}/ifss/starboard"/>
-            </sensor>
-            <world_transform rpy="${rpy}" xyz="${xyz}"/>
-        </robot>
-    </xacro:macro>
+    <xacro:include filename="$(find alpha_stonefish)/description/alpha_v1-1.scn.xacro"/>
+    <xacro:include filename="$(find alpha_stonefish)/description/alpha_v1-2.scn.xacro"/>
 </scenario>

File: alpha_stonefish/scenarios/ocean.scn.xacro (robot description, xacro)
@@ -10,5 +10,5 @@
     <xacro:arg name="robot_name" default="changeme"/>
     <xacro:include filename="$(find alpha_stonefish)/description/alpha.scn.xacro"/>
-    <xacro:alpha robot_name="$(arg robot_name)" xyz="0.0 0.0 0.0" rpy="0.0 0.0 0.0"/>
+    <xacro:alpha_v1-2 robot_name="$(arg robot_name)" xyz="0.0 0.0 0.0" rpy="0.0 0.0 0.0"/>
     <environment>
         <ned latitude="41" longitude="71"/>

File: alpha_stonefish/scenarios/ocean_multi_agent.scn.xacro (robot description, xacro)
@@ -9,8 +9,8 @@
 <scenario xmlns:xacro="http://ros.org/wiki/xacro">
     <xacro:include filename="$(find alpha_stonefish)/description/alpha.scn.xacro"/>
-    <xacro:alpha robot_name="bill" xyz="0.0 0.0 0.0" rpy="0.0 0.0 0.0"/>
-    <xacro:alpha robot_name="lin" xyz="5.0 0.0 0.0" rpy="0.0 0.0 0.0"/>
-    <xacro:alpha robot_name="emir" xyz="5.0 5.0 0.0" rpy="0.0 0.0 0.0"/>
-    <xacro:alpha robot_name="mingxi" xyz="0.0 5.0 0.0" rpy="0.0 0.0 0.0"/>
+    <xacro:alpha_v1-1 robot_name="bill" xyz="0.0 0.0 0.0" rpy="0.0 0.0 0.0"/>
+    <xacro:alpha_v1-1 robot_name="lin" xyz="5.0 0.0 0.0" rpy="0.0 0.0 0.0"/>
+    <xacro:alpha_v1-1 robot_name="emir" xyz="5.0 5.0 0.0" rpy="0.0 0.0 0.0"/>
+    <xacro:alpha_v1-1 robot_name="mingxi" xyz="0.0 5.0 0.0" rpy="0.0 0.0 0.0"/>
     <environment>
         <ned latitude="41" longitude="71"/>

File: alpha_stonefish/scenarios/tank.scn.xacro (robot description, xacro)
@@ -10,4 +10,5 @@
     <xacro:arg name="robot_name" default="changeme"/>
     <xacro:include filename="$(find alpha_stonefish)/description/alpha.scn.xacro"/>
+    <xacro:alpha_v1-1 robot_name="$(arg robot_name)" xyz="0.0 0.0 0.0" rpy="0.0 0.0 0.0"/>
     <environment>
         <ned latitude="41.7777" longitude="3.0333"/>

Commit message: chore: remove new model vehicle

File: alpha_stonefish/description/alpha.scn.xacro (robot description, xacro)
@@ -1,4 +1,168 @@
+<?xml version="1.0"?>
+<!--
+    This file is part of ALPHA AUV project.
+    Author: Emir Cem Gezer
+    Email: emircem@uri.edu;emircem.gezer@gmail.com
+    Year: 2022
+    Copyright (C) 2022 Smart Ocean Systems Laboratory
+-->
 <scenario xmlns:xacro="http://ros.org/wiki/xacro">
-    <xacro:include filename="$(find alpha_stonefish)/description/alpha_v1-1.scn.xacro"/>
-    <xacro:include filename="$(find alpha_stonefish)/description/alpha_v1-2.scn.xacro"/>
+    <xacro:include filename="$(find alpha_stonefish)/description/looks.scn.xacro"/>
+    <xacro:include filename="$(find alpha_stonefish)/description/materials.scn.xacro"/>
+    <xacro:macro name="alpha" params="xyz rpy robot_name">
+        <robot name="${robot_name}" fixed="false" self_collisions="false">
+            <base_link name="Vehicle" type="compound" physics="submerged">
+                <external_part name="Hull" type="model" physics="submerged" buoyant="false">
+                    <physical>
+                        <mesh filename="hull_phy_reduced.obj" scale="1.0"/>
+                        <origin rpy="0.0 0.0 0.0" xyz="0.0 0.0 0.0"/>
+                    </physical>
+                    <visual>
+                        <mesh filename="hull.obj" scale="1.0"/>
+                        <origin rpy="0.0 0.0 0.0" xyz="0.0 0.0 0.0"/>
+                    </visual>
+                    <material name="Vehicle"/>
+                    <look name="yellow"/>
+                    <mass value="24.8"/>
+                    <compound_transform rpy="0.0 0.0 0.0" xyz="0.0 0.0 0.0"/>
+                    <cg xyz="-0.65 0.0 0.1" rpy="0.0 0.0 0.0"/>
+                </external_part>
+                <internal_part name="Foam" type="cylinder" physics="floating" buoyant="true">
+                    <dimensions radius="0.1" height="1.0"/>
+                    <origin rpy="0.0 0.0 0.0" xyz="0.0 0.0 0.0"/>
+                    <material name="Foam"/>
+                    <mass value="6.0"/>
+                    <look name="grey"/>
+                    <compound_transform rpy="0.0 1.571 0.0" xyz="-0.65 0.0 -0.05"/>
+                </internal_part>
+                <external_part name="Mast" type="model" physics="submerged">
+                    <physical>
+                        <mesh filename="mast.obj" scale="0.001"/>
+                        <origin rpy="-1.571 0.0 1.571"  xyz="-1.0 0.0 0.0"/>
+                    </physical>
+                    <visual>
+                        <mesh filename="mast.obj" scale="0.001"/>
+                        <origin rpy="-1.571 0.0 1.571" xyz="-1.0 0.0 0.0"/>
+                    </visual>
+                    <material name="Resin"/>
+                    <look name="white"/>
+                    <compound_transform rpy="0.0 0.0 0.0" xyz="0.0 0.0 0.0"/>
+                </external_part>
+                <external_part name="ThrusterDuctSurge" type="model" physics="submerged" buoyant="false">
+                    <physical>
+                        <mesh filename="duct.obj" scale="0.0015"/>
+                        <origin rpy="0.0 1.571 0.0" xyz="-1.325 0.0 0.0"/>
+                    </physical>
+                    <visual>
+                        <mesh filename="duct.obj" scale="0.0015"/>
+                        <origin rpy="0.0 1.571 0.0" xyz="-1.325 0.0 0.0"/>
+                    </visual>
+                    <material name="Neutral"/>
+                    <look name="black"/>
+                    <compound_transform rpy="0.0 0.0 0.0" xyz="0.0 0.0 0.0"/>
+                </external_part>
+            </base_link>
+            <actuator name="ThrusterHeaveStern" type="thruster">
+                <link name="Vehicle"/>
+                <origin rpy="0.0 -1.571 0.0" xyz="-1.0956 0.0 0.0"/>
+                <specs thrust_coeff="0.4315" thrust_coeff_backward="0.3404" torque_coeff="0.01" max_rpm="3000.0"/>
+                <propeller diameter="0.08" right="true">
+                    <mesh filename="prop.obj" scale="1.0"/>
+                    <material name="Neutral"/>
+                    <look name="white"/>
+                </propeller>
+                <ros_subscriber topic="/${robot_name}/control/thruster/heave_stern"/>
+            </actuator>
+            <actuator name="ThrusterHeaveBow" type="thruster">
+                <link name="Vehicle"/>
+                <origin rpy="0.0 -1.571 0.0" xyz="-0.2857 0.0 0.0"/>
+                <specs thrust_coeff="0.4315" thrust_coeff_backward="0.3404" torque_coeff="0.01" max_rpm="3000.0"/>
+                <propeller diameter="0.08" right="true">
+                    <mesh filename="prop.obj" scale="1.0"/>
+                    <material name="Neutral"/>
+                    <look name="white"/>
+                </propeller>
+                <ros_subscriber topic="/${robot_name}/control/thruster/heave_bow"/>
+            </actuator>
+            <actuator name="ThrusterSwayBow" type="thruster">
+                <link name="Vehicle"/>
+                <origin rpy="0.0 0.0 -1.571" xyz="-0.171 0.0 0.0"/>
+                <specs thrust_coeff="0.4315" thrust_coeff_backward="0.3404" torque_coeff="0.01" max_rpm="3000.0"/>
+                <propeller diameter="0.08" right="true">
+                    <mesh filename="prop.obj" scale="1.0"/>
+                    <material name="Neutral"/>
+                    <look name="white"/>
+                </propeller>
+                <ros_subscriber topic="/${robot_name}/control/thruster/sway_bow"/>
+            </actuator>
+            <actuator name="ThrusterSurge" type="thruster">
+                <link name="Vehicle"/>
+                <origin rpy="0.0 0.0 0.0" xyz="-1.325 0.0 0.0"/>
+                <specs thrust_coeff="1.7568" thrust_coeff_backward="1.0882" torque_coeff="0.01" max_rpm="3000.0"/>
+                <propeller diameter="0.08" right="true">
+                    <origin rpy="1.571 0.0 0.0" xyz="0.0 0.0 0.0"/>
+                    <mesh filename="prop.obj" scale="1.5"/>
+                    <material name="Neutral"/>
+                    <look name="white"/>
+                </propeller>
+                <ros_subscriber topic="/${robot_name}/control/thruster/surge"/>
+            </actuator>
+            <sensor name="pressure" type="pressure" rate="5.0">
+                <link name="Vehicle"/>
+                <origin rpy="0.0 0.0 0.0" xyz="-1.20 0.0 0.0"/>
+                <noise pressure="5.0"/>
+                <ros_publisher topic="/${robot_name}/pressure"/>
+            </sensor>
+            <sensor name="dvl" type="dvl" rate="5.0">
+                <link name="Vehicle"/>
+                <origin rpy="3.1416 0.0 0.0" xyz="-0.75 0.0 0.10"/>
+                <specs beam_angle="30.0"/>
+                <range velocity="9.0 9.0 9.0" altitude_min="0.05" altitude_max="200.0"/>
+                <noise velocity="0.0015" altitude="0.001"/>
+                <ros_publisher topic="/${robot_name}/dvl/twist" altitude_topic="/${robot_name}/dvl/altitude"/>
+            </sensor>
+            <sensor name="imu" type="imu" rate="20.0">
+                <link name="Vehicle"/>
+                <origin rpy="0.0 0.0 0.0" xyz="-0.65 0.0 0.0"/>
+                <noise angle="0.000001745" angular_velocity="0.00001745"/>
+                <ros_publisher topic="/${robot_name}/imu/stonefish/data"/>
+            </sensor>
+            <sensor name="gps" type="gps" rate="1.0">
+                <link name="Vehicle"/>
+                <origin rpy="0.0 0.0 0.0" xyz="-0.54 0.0 -0.2"/>
+                <noise ned_position="0.5"/>
+                <ros_publisher topic="/${robot_name}/gps/fix"/>
+            </sensor>
+            <sensor name="multibeam" rate="50.0" type="multibeam">
+                <specs fov="90.0" steps="64"/>
+                <range distance_min="0.5" distance_max="200.0"/>
+                <noise distance="0.0"/>
+                <history samples="1"/>
+                <origin xyz="0.0 0.0 0.2" rpy="0.0 -1.0471975511965976 0.0"/>
+                <link name="Vehicle"/>
+                <ros_publisher topic="/${robot_name}/mbs/data"/>
+            </sensor>
+            <sensor name="ifss_port_swath" rate="10.0" type="multibeam">
+                <specs fov="53.0" steps="64"/>
+                <range distance_min="0.1" distance_max="150.0"/>
+                <noise distance="0.0"/>
+                <history samples="1"/>
+                <origin xyz="-0.75 -0.0762 0.2" rpy="-1.5708 -2.35619 1.5708"/>
+                <link name="Vehicle"/>
+                <pcl_topic topic="/${robot_name}/ifss/port/pcl"/>
+                <ros_publisher topic="/${robot_name}/ifss/port"/>
+            </sensor>
+            <sensor name="ifss_starboard_swath" rate="10.0" type="multibeam">
+                <specs fov="53.0" steps="64"/>
+                <range distance_min="0.1" distance_max="150.0"/>
+                <noise distance="0.0"/>
+                <history samples="1"/>
+                <origin xyz="-0.75 0.0762 0.2" rpy="1.5708 -2.35619 -1.5708"/>
+                <link name="Vehicle"/>
+                <pcl_topic topic="/${robot_name}/ifss/starboard/pcl"/>
+                <ros_publisher topic="/${robot_name}/ifss/starboard"/>
+            </sensor>
+            <world_transform rpy="${rpy}" xyz="${xyz}"/>
+        </robot>
+    </xacro:macro>
 </scenario>

File: alpha_stonefish/scenarios/ocean.scn.xacro (robot description, xacro)
@@ -10,5 +10,5 @@
     <xacro:arg name="robot_name" default="changeme"/>
     <xacro:include filename="$(find alpha_stonefish)/description/alpha.scn.xacro"/>
-    <xacro:alpha_v1-1 robot_name="$(arg robot_name)" xyz="0.0 0.0 0.0" rpy="0.0 0.0 0.0"/>
+    <xacro:alpha robot_name="$(arg robot_name)" xyz="0.0 0.0 0.0" rpy="0.0 0.0 0.0"/>
     <environment>
         <ned latitude="41" longitude="71"/>

File: alpha_stonefish/scenarios/ocean_multi_agent.scn.xacro (robot description, xacro)
@@ -9,8 +9,8 @@
 <scenario xmlns:xacro="http://ros.org/wiki/xacro">
     <xacro:include filename="$(find alpha_stonefish)/description/alpha.scn.xacro"/>
-    <xacro:alpha_v1-1 robot_name="bill" xyz="0.0 0.0 0.0" rpy="0.0 0.0 0.0"/>
-    <xacro:alpha_v1-1 robot_name="lin" xyz="5.0 0.0 0.0" rpy="0.0 0.0 0.0"/>
-    <xacro:alpha_v1-1 robot_name="emir" xyz="5.0 5.0 0.0" rpy="0.0 0.0 0.0"/>
-    <xacro:alpha_v1-1 robot_name="mingxi" xyz="0.0 5.0 0.0" rpy="0.0 0.0 0.0"/>
+    <xacro:alpha robot_name="bill" xyz="0.0 0.0 0.0" rpy="0.0 0.0 0.0"/>
+    <xacro:alpha robot_name="lin" xyz="5.0 0.0 0.0" rpy="0.0 0.0 0.0"/>
+    <xacro:alpha robot_name="emir" xyz="5.0 5.0 0.0" rpy="0.0 0.0 0.0"/>
+    <xacro:alpha robot_name="mingxi" xyz="0.0 5.0 0.0" rpy="0.0 0.0 0.0"/>
     <environment>
         <ned latitude="41" longitude="71"/>

File: alpha_stonefish/scenarios/tank.scn.xacro (robot description, xacro)
@@ -10,5 +10,5 @@
     <xacro:arg name="robot_name" default="changeme"/>
     <xacro:include filename="$(find alpha_stonefish)/description/alpha.scn.xacro"/>
-    <xacro:alpha_v1-1 robot_name="$(arg robot_name)" xyz="0.0 0.0 0.0" rpy="0.0 0.0 0.0"/>
+    <xacro:alpha robot_name="$(arg robot_name)" xyz="0.0 0.0 0.0" rpy="0.0 0.0 0.0"/>
     <environment>
         <ned latitude="41.7777" longitude="3.0333"/>
